File: Hardware/FlightController/DronePCB.kicad_pcb (KiCad board)
At the start: 2 copper layers, 53.1 x 93.3 mm, 15 parts, among them U1 ESP32-DEVKIT-V1

Commit message: PCB Drone et manette finis avec gerbers générés
Parts:
- NRF24L01: footprint Connector_PinHeader_2.00mm:PinHeader_2x04_P2.00mm_Vertical -> Connector_PinHeader_2.54mm:PinHeader_2x04_P2.54mm_Vertical
- R3: value 100k -> 100000
- R4: value 15k -> 15000
- moved NRF24L01 1.56 mm to (39.0, 106.5)
Routing:
- net GND: track 11.5 -> 34.6 mm, vias 26 -> 33
- net NRF_CE: track 65.7 -> 68.7 mm
- net NRF_CSN: track 73.0 -> 72.0 mm
- net SCK: track 54.0 -> 55.0 mm

Commit message: Correction Drone pinout et génération gerber
Connections:
- U1 pad 21: Moteur3 -> unconnected-(U1-D32-Pad21)
- U1 pad 24: SDA_1 -> Moteur3
- U1 pad 25: unconnected-(U1-D27-Pad25) -> Moteur2
- U1 pad 26: Moteur2 -> SDA_1
Routing:
- net SDA_1: track 40.0 -> 45.1 mm
- net Moteur3: track 52.0 -> 54.7 mm
- net Moteur2: track 32.0 -> 34.5 mm
- net NRF_CSN: track 72.0 -> 74.1 mm
- net MISO: track 57.2 -> 58.7 mm
Changed lines of the file:
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@@
 	(net 27 "unconnected-(U1-RX2-Pad6)")
 	(net 28 "unconnected-(U1-EN-Pad16)")
-	(net 29 "unconnected-(U1-D27-Pad25)")
+	(net 29 "unconnected-(U1-D32-Pad21)")
 	(net 30 "unconnected-(U1-D2-Pad4)")
 	(net 31 "unconnected-(U1-TX2-Pad7)")
@@
 		(tags "Through hole pin header THT 1x07 2.54mm single row")
 		(property "Reference" "SIGNAUX"
-			(at 1.1 -5.56 180)
+			(at 0.3 -5.56 180)
 			(layer "F.SilkS")
 			(effects
@@
 			(layer "F.Fab")
 		)
-		(fp_text user "${REFERENCE}"
-			(at 0 7.62 0)
-			(layer "F.Fab")
-			(effects
-				(font
-					(size 1 1)
-					(thickness 0.15)
-				)
-			)
-		)
 		(pad "1" thru_hole rect
 			(at 0 0 90)
@@
 			(layers "*.Cu" "*.Mask")
 			(remove_unused_layers no)
-			(net 15 "Moteur3")
+			(net 29 "unconnected-(U1-D32-Pad21)")
 			(pinfunction "D32")
-			(pintype "bidirectional")
+			(pintype "bidirectional+no_connect")
 			(solder_mask_margin 0.102)
 		)
@@
 			(layers "*.Cu" "*.Mask")
 			(remove_unused_layers no)
-			(net 8 "SDA_1")
+			(net 15 "Moteur3")
 			(pinfunction "D26")
 			(pintype "bidirectional")
@@
 			(layers "*.Cu" "*.Mask")
 			(remove_unused_layers no)
-			(net 29 "unconnected-(U1-D27-Pad25)")
+			(net 14 "Moteur2")
 			(pinfunction "D27")
-			(pintype "bidirectional+no_connect")
+			(pintype "bidirectional")
 			(solder_mask_margin 0.102)
 		)
@@
 			(layers "*.Cu" "*.Mask")
 			(remove_unused_layers no)
-			(net 14 "Moteur2")
+			(net 8 "SDA_1")
 			(pinfunction "D14")
 			(pintype "bidirectional")
@@
 			(layer "F.Fab")
 		)
-		(fp_text user "${REFERENCE}"
-			(at 0 11.43 0)
-			(layer "F.Fab")
-			(effects
-				(font
-					(size 1 1)
-					(thickness 0.15)
-				)
-			)
-		)
 		(pad "1" thru_hole rect
 			(at 0 0 270)
@@
 		(tags "Through hole pin header THT 2x04 2.54mm double row")
 		(property "Reference" "NRF24L01"
-			(at -1.5 15.04 180)
+			(at -1.2 13.74 180)
 			(layer "F.SilkS")
 			(effects
@@
 			(layer "F.Fab")
 		)
-		(fp_text user "${REFERENCE}"
-			(at 1.27 3.81 180)
-			(layer "F.Fab")
-			(effects
-				(font
-					(size 1 1)
-					(thickness 0.15)
-				)
-			)
-		)
 		(pad "1" thru_hole rect
 			(at 0 0 90)
@@
 	)
 	(segment
+		(start 25.9 67.3)
+		(end 25.9 67.1)
+		(width 0.2)
+		(layer "F.Cu")
+		(net 2)
+	)
+	(segment
+		(start 25.7 61.2)
+		(end 25.6 61.1)
+		(width 0.2)
+		(layer "F.Cu")
+		(net 2)
+	)
+	(segment
+		(start 25.7 66.9)
+		(end 25.7 61.2)
+		(width 0.2)
+		(layer "F.Cu")
+		(net 2)
+	)
+	(segment
 		(start 33.8 91.2)
 		(end 35 90)
@@
 		(net 2)
 	)
+	(segment
+		(start 25.9 67.1)
+		(end 25.7 66.9)
+		(width 0.2)
+		(layer "F.Cu")
+		(net 2)
+	)
 	(via
 		(at 65 75)
@@
 	)
 	(via
+		(at 25.9 67.3)
+		(size 0.6)
+		(drill 0.3)
+		(layers "F.Cu" "B.Cu")
+		(free yes)
+		(net 2)
+	)
+	(via
 		(at 60.5 38.5)
 		(size 0.6)
@@
 	)
 	(via
-		(at 29.2 107.2)
+		(at 25.6 61.1)
 		(size 0.6)
 		(drill 0.3)
@@
 	)
 	(via
-		(at 20 35)
+		(at 29.2 107.2)
 		(size 0.6)
 		(drill 0.3)
@@
 	)
 	(via
-		(at 37.5 53)
+		(at 20 35)
 		(size 0.6)
 		(drill 0.3)
@@
 	)
 	(via
-		(at 65.5 44.5)
+		(at 37.5 53)
 		(size 0.6)
 		(drill 0.3)
@@
 	)
 	(via
-		(at 30.9 96.1)
+		(at 65.5 44.5)
 		(size 0.6)
 		(drill 0.3)
@@
 	)
 	(via
-		(at 44.5 41)
+		(at 30.9 96.1)
 		(size 0.6)
 		(drill 0.3)
@@
 		(net 2)
 	)
-	(via
-		(at 48.2 36.6)
-		(size 0.6)
-		(drill 0.3)
-		(layers "F.Cu" "B.Cu")
-		(free yes)
-		(net 2)
-	)
 	(segment
 		(start 62.7 82.7)
@@
 	)
 	(segment
-		(start 48.2 36.6)
-		(end 44.5 40.3)
-		(width 0.2)
-		(layer "B.Cu")
-		(net 2)
-	)
-	(segment
-		(start 44.5 40.3)
-		(end 44.5 41)
-		(width 0.2)
-		(layer "B.Cu")
-		(net 2)
-	)
-	(segment
 		(start 31.3 105.1)
 		(end 29.2 107.2)
@@
 	)
 	(segment
-		(start 52.2 54.225)
-		(end 52.2 78.4)
+		(start 53.2 79.2)
+		(end 57.02 79.2)
 		(width 0.2)
 		(layer "F.Cu")
@@
 	)
 	(segment
-		(start 52.2 78.4)
-		(end 53 79.2)
+		(start 57.02 79.2)
+		(end 61.6 74.62)
 		(width 0.2)
 		(layer "F.Cu")
@@
 	)
 	(segment
-		(start 55.2 51.225)
-		(end 52.2 54.225)
+		(start 55.2 46.145)
+		(end 52.1 49.245)
 		(width 0.2)
 		(layer "F.Cu")
@@
 	)
 	(segment
-		(start 53 79.2)
-		(end 57.02 79.2)
+		(start 52.1 78.1)
+		(end 53.2 79.2)
 		(width 0.2)
 		(layer "F.Cu")
@@
 	)
 	(segment
-		(start 57.02 79.2)
-		(end 61.6 74.62)
+		(start 52.1 49.245)
+		(end 52.1 78.1)
 		(width 0.2)
 		(layer "F.Cu")
@@
 	)
 	(segment
-		(start 25 97.3)
-		(end 25.9 98.2)
+		(start 23.2 65.445)
+		(end 23.2 95.5)
 		(width 0.2)
 		(layer "B.Cu")
@@
 	)
 	(segment
-		(start 25 63.645)
-		(end 25 97.3)
+		(start 23.2 95.5)
+		(end 25.9 98.2)
 		(width 0.2)
 		(layer "B.Cu")
@@
 	(segment
 		(start 29.8 58.845)
-		(end 25 63.645)
+		(end 23.2 65.445)
 		(width 0.2)
 		(layer "B.Cu")
@@
 	)
 	(segment
-		(start 24.2 98.7)
-		(end 34 108.5)
+		(start 29.8 53.765)
+		(end 21.6 61.965)
 		(width 0.2)
 		(layer "F.Cu")
@@
 	)
 	(segment
-		(start 34 108.5)
-		(end 42.04 108.5)
+		(start 21.6 61.965)
+		(end 21.6 96.1)
 		(width 0.2)
 		(layer "F.Cu")
@@
 	)
 	(segment
-		(start 29.8 53.765)
-		(end 24.2 59.365)
+		(start 34 108.5)
+		(end 42.04 108.5)
 		(width 0.2)
 		(layer "F.Cu")
@@
 	)
 	(segment
-		(start 24.2 59.365)
-		(end 24.2 98.7)
+		(start 21.6 96.1)
+		(end 34 108.5)
 		(width 0.2)
 		(layer "F.Cu")
@@
 	)
 	(segment
-		(start 39.64 30.585)
-		(end 55.2 46.145)
+		(start 39.64 20.6)
+		(end 39.64 33.125)
 		(width 0.3)
-		(layer "F.Cu")
+		(layer "B.Cu")
 		(net 14)
 	)
 	(segment
-		(start 39.64 20.6)
-		(end 39.64 30.585)
+		(start 39.64 33.125)
+		(end 55.2 48.685)
 		(width 0.3)
-		(layer "F.Cu")
+		(layer "B.Cu")
 		(net 14)
 	)
 	(segment
-		(start 58.5 36)
-		(end 56 33.5)
+		(start 55.2 51.225)
+		(end 56.675 51.225)
 		(width 0.3)
 		(layer "B.Cu")
@@
 	)
 	(segment
-		(start 56 33.5)
-		(end 50 33.5)
+		(start 56.675 51.225)
+		(end 57.2 50.7)
 		(width 0.3)
 		(layer "B.Cu")
@@
 	)
 	(segment
-		(start 58.5 55.545)
-		(end 58.5 36)
+		(start 55.5 18.3)
+		(end 39.4 18.3)
 		(width 0.3)
 		(layer "B.Cu")
@@
 	)
 	(segment
-		(start 55.2 58.845)
-		(end 58.5 55.545)
+		(start 57.2 50.7)
+		(end 57.2 20)
 		(width 0.3)
 		(layer "B.Cu")
@@
 	)
 	(segment
-		(start 50 33.5)
+		(start 39.4 18.3)
 		(end 37.1 20.6)
 		(width 0.3)
@@
 	)
 	(segment
+		(start 57.2 20)
+		(end 55.5 18.3)
+		(width 0.3)
+		(layer "B.Cu")
+		(net 15)
+	)
+	(segment
 		(start 42.18 20.6)
 		(end 42.18 28.045)
@@
 	)
 	(segment
-		(start 49.12 29.905)
-		(end 55.2 35.985)
-		(width 0.4)
-		(layer "F.Cu")
-		(net 17)
-	)
-	(segment
-		(start 44.72 20.6)
-		(end 49.12 25)
+		(start 44.72 25.505)
+		(end 44.72 20.6)
 		(width 0.4)
 		(layer "F.Cu")
@@
 	)
 	(segment
-		(start 49.12 25)
-		(end 49.12 29.905)
+		(start 55.2 35.985)
+		(end 44.72 25.505)
 		(width 0.4)
 		(layer "F.Cu")
